Commit message: custom vehicle and sensor packages working

File: sensor_kit/nuway_sensor_kit_launch/nuway_sensor_kit_description/urdf/sensor_kit.xacro (robot description, xacro)
@@ -85,5 +85,6 @@
     <!-- Cameras -->
     <xacro:monocular_camera_macro
-      name="camera_front/camera"
+	  namespace="camera_front"
+	  name="camera_front/camera"
       parent="sensor_kit_base_link"
       x="${calibration['sensor_kit_base_link']['camera_front']['x']}"
@@ -96,4 +97,5 @@
     />
     <xacro:monocular_camera_macro
+      namespace="camera_rear"
       name="camera_rear/camera"
       parent="sensor_kit_base_link"
@@ -108,4 +110,5 @@
     <!-- IMU -->
     <xacro:imu_macro
+      namespace=""
       name="tamagawa/imu"
       parent="sensor_kit_base_link"

File: vehicle/nuway_vehicle_launch/nuway_vehicle_description/urdf/vehicle.xacro (robot description, xacro)
@@ -2,5 +2,5 @@
 <robot xmlns:xacro="http://ros.org/wiki/xacro">
   <!-- load parameter -->
-  <xacro:property name="vehicle_info" value="${xacro.load_yaml('$(find description)/config/vehicle_info.param.yaml')}"/>
+  <xacro:property name="vehicle_info" value="${xacro.load_yaml('$(find nuway_vehicle_description)/config/vehicle_info.param.yaml')}"/>
   <!-- vehicle body -->
   <link name="base_link">

Commit message: Updated a few things

File: sensor_kit/nuway_sensor_kit_launch/nuway_sensor_kit_description/urdf/sensor_kit.xacro (robot description, xacro)
@@ -43,44 +43,4 @@
       />
     </xacro:VLP-16>
-    <xacro:VLS-128 parent="sensor_kit_base_link" name="lidar_safety_front_left" topic="/points_raw" hz="10" samples="220" gpu="$(arg gpu)">
-      <origin
-        xyz="${calibration['sensor_kit_base_link']['lidar_safety_front_left']['x']}
-             ${calibration['sensor_kit_base_link']['lidar_safety_front_left']['y']}
-             ${calibration['sensor_kit_base_link']['lidar_safety_front_left']['z']}"
-        rpy="${calibration['sensor_kit_base_link']['lidar_safety_front_left']['roll']}
-             ${calibration['sensor_kit_base_link']['lidar_safety_front_left']['pitch']}
-             ${calibration['sensor_kit_base_link']['lidar_safety_front_left']['yaw']}"
-      />
-    </xacro:VLS-128>
-    <xacro:VLS-128 parent="sensor_kit_base_link" name="lidar_safety_front_right" topic="/points_raw" hz="10" samples="220" gpu="$(arg gpu)">
-      <origin
-        xyz="${calibration['sensor_kit_base_link']['lidar_safety_front_right']['x']}
-             ${calibration['sensor_kit_base_link']['lidar_safety_front_right']['y']}
-             ${calibration['sensor_kit_base_link']['lidar_safety_front_right']['z']}"
-        rpy="${calibration['sensor_kit_base_link']['lidar_safety_front_right']['roll']}
-             ${calibration['sensor_kit_base_link']['lidar_safety_front_right']['pitch']}
-             ${calibration['sensor_kit_base_link']['lidar_safety_front_right']['yaw']}"
-      />
-    </xacro:VLS-128>
-    <xacro:VLS-128 parent="sensor_kit_base_link" name="lidar_safety_rear_left" topic="/points_raw" hz="10" samples="220" gpu="$(arg gpu)">
-      <origin
-        xyz="${calibration['sensor_kit_base_link']['lidar_safety_rear_left']['x']}
-             ${calibration['sensor_kit_base_link']['lidar_safety_rear_left']['y']}
-             ${calibration['sensor_kit_base_link']['lidar_safety_rear_left']['z']}"
-        rpy="${calibration['sensor_kit_base_link']['lidar_safety_rear_left']['roll']}
-             ${calibration['sensor_kit_base_link']['lidar_safety_rear_left']['pitch']}
-             ${calibration['sensor_kit_base_link']['lidar_safety_rear_left']['yaw']}"
-      />
-    </xacro:VLS-128>
-    <xacro:VLS-128 parent="sensor_kit_base_link" name="lidar_safety_rear_right" topic="/points_raw" hz="10" samples="220" gpu="$(arg gpu)">
-      <origin
-        xyz="${calibration['sensor_kit_base_link']['lidar_safety_rear_right']['x']}
-             ${calibration['sensor_kit_base_link']['lidar_safety_rear_right']['y']}
-             ${calibration['sensor_kit_base_link']['lidar_safety_rear_right']['z']}"
-        rpy="${calibration['sensor_kit_base_link']['lidar_safety_rear_right']['roll']}
-             ${calibration['sensor_kit_base_link']['lidar_safety_rear_right']['pitch']}
-             ${calibration['sensor_kit_base_link']['lidar_safety_rear_right']['yaw']}"
-      />
-    </xacro:VLS-128>
     <!-- Cameras -->
     <xacro:monocular_camera_macro
